Commit message: Clean simulator working

File: kuka_pentomino/src/ec2_bringup/description/miiwa/miiwa.urdf.xacro (robot description, xacro)
@@ -125,10 +125,10 @@
     />
   </xacro:mako_3d>
-  <xacro:mako_3d
-    name="cameras_tcp_rect/right"
-    parent_link="cameras_tcp_rect/left_link"
-  >
-    <origin xyz="${mako_3d_hand_relative_offset} 0 0" rpy="0.0 0.0 0.0"/>
-  </xacro:mako_3d>
+  <!-- <xacro:mako_3d -->
+  <!--   name="cameras_tcp_rect/right" -->
+  <!--   parent_link="cameras_tcp_rect/left_link" -->
+  <!-- > -->
+  <!--   <origin xyz="${mako_3d_hand_relative_offset} 0 0" rpy="0.0 0.0 0.0"/> -->
+  <!-- </xacro:mako_3d> -->
   <xacro:manta
     name="cameras_pan_tilt/left"
@@ -140,10 +140,10 @@
     />
   </xacro:manta>
-  <xacro:manta
-    name="cameras_pan_tilt/right"
-    parent_link="cameras_pan_tilt/left_link"
-  >
-    <origin xyz="${manta_mast_relative_offset} 0 0" rpy="0.0 0.0 0.0"/>
-  </xacro:manta>
+  <!-- <xacro:manta -->
+  <!--   name="cameras_pan_tilt/right" -->
+  <!--   parent_link="cameras_pan_tilt/left_link" -->
+  <!-- > -->
+    <!-- <origin xyz="${manta_mast_relative_offset} 0 0" rpy="0.0 0.0 0.0"/> -->
+  <!-- </xacro:manta> -->
     <!-- additions for gazebo -->
   <xacro:mako_depth_camera_gazebo

File: kuka_pentomino/src/ec2_bringup/description/miiwa/miiwa_base.gazebo.xacro (robot description, xacro)
@@ -34,5 +34,5 @@
          </image>
        </camera>
-       <plugin name="depth_camera_controller" filename="libgazebo_ros_depth_camera.so">
+       <plugin name="depth_camera_controller" filename="libgazebo_ros_openni_kinect.so">
          <alwaysOn>true</alwaysOn>
          <updateRate>${rate}</updateRate>
@@ -42,5 +42,5 @@
          <pointCloudTopicName>point_cloud</pointCloudTopicName>
          <depthImageTopicName>depth</depthImageTopicName>
-         <depthImageCameraInfoTopicName>camera_info</depthImageCameraInfoTopicName>
+         <!-- <depthImageCameraInfoTopicName>camera_info</depthImageCameraInfoTopicName> -->
          <pointCloudCutoff>0.10</pointCloudCutoff>
          <frameName>tcp_stereo_left_rect</frameName>
@@ -66,5 +66,5 @@
          </image>
        </camera>
-       <plugin name="depth_camera_controller" filename="libgazebo_ros_depth_camera.so">
+       <plugin name="depth_camera_controller" filename="libgazebo_ros_openni_kinect.so">
          <alwaysOn>true</alwaysOn>
          <updateRate>${rate}</updateRate>
@@ -74,5 +74,5 @@
          <pointCloudTopicName>point_cloud</pointCloudTopicName>
          <depthImageTopicName>depth</depthImageTopicName>
-         <depthImageCameraInfoTopicName>camera_info</depthImageCameraInfoTopicName>
+         <!-- <depthImageCameraInfoTopicName>camera_info</depthImageCameraInfoTopicName> -->
          <pointCloudCutoff>0.4</pointCloudCutoff>
          <frameName>${parent_link}</frameName>
